File: Gate_drive_module_Si8285/Gate_driver.kicad_pcb (KiCad board)
At the start: 2 copper layers, 34 parts, among them J1 CONN_01X10, J2 CONN_01X04, J3 CONN_01X03, J4 CONN_01X03, J5 CONN_01X03, U1 Si8285, U2 Mornsun_QA01C

Commit message: PCB layout nearly finished, comments are welcome
Parts:
- removed D5, D6: GREEN PWR LED, LEDs:LED_0805_HandSoldering
- added C12: 100n, Capacitors_SMD:C_0805_HandSoldering, F.Cu at (147.4, 124.9)
- C10: value 100n -> 10u
- C3, C5: footprint Capacitors_SMD:C_1812_HandSoldering -> Capacitors_SMD:CP_Elec_6.3x7.7
- C4: value 100u -> 100n; footprint Capacitors_SMD:C_1812_HandSoldering -> Capacitors_SMD:C_0805_HandSoldering
- C6: value 100p -> 100u; footprint Capacitors_SMD:C_0805_HandSoldering -> Capacitors_SMD:CP_Elec_6.3x7.7
- C7: value 10u -> 390p
- D3, D4: footprint Diodes_SMD:D_SMA_Handsoldering -> LEDs:LED_0805_HandSoldering
- R4, R5: footprint Resistors_SMD:R_0805_HandSoldering -> Resistors_SMD:R_1206_HandSoldering; moved to B.Cu
- U2: footprint mornsun:QA01C -> Mornsun:QA01C
- moved C7 55.1 mm to (154.7, 117.7), turned to 180 degrees
- moved C8 52.2 mm to (152.4, 122.7), turned to 270 degrees
- moved R6 50.1 mm to (159.6, 117.7), turned to 180 degrees
- moved TP1 48.3 mm to (160.9, 111.6)
- moved C9 44.9 mm to (145.2, 120.1), turned to 270 degrees
- moved R4 43.2 mm to (166.2, 121.0), turned to 180 degrees
- moved J5 41.1 mm to (181.4, 138.4)
- moved C4 40.3 mm to (116.5, 137.4), turned to 90 degrees
- moved J4 40.1 mm to (174.8, 126.4)
- moved C11 36.0 mm to (147.4, 120.1), turned to 270 degrees
- moved R5 35.2 mm to (166.2, 124.3), turned to 180 degrees
- moved R9 32.5 mm to (172.8, 135.7), turned to 90 degrees
- moved D2 32.2 mm to (167.1, 116.3), turned to 180 degrees
- moved C10 32.0 mm to (145.2, 124.9), turned to 270 degrees
- moved R8 31.1 mm to (169.2, 135.6), turned to 270 degrees
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Connections:
- C10 pad 1: VCC_ISO -> GND_ISO
- C10 pad 2: GND_ISO -> VEE_ISO
- C11 pad 1: GND_ISO -> VCC_ISO
- C11 pad 2: VEE_ISO -> GND_ISO
- C4 pad 1: VCC_ISO -> +15V
- C4 pad 2: GND_ISO -> GND
- C5 pad 1: GND_ISO -> VCC_ISO
- C5 pad 2: VEE_ISO -> GND_ISO
- C6 pad 1: Net-(C6-Pad1) -> GND_ISO
- C6 pad 2: GND_ISO -> VEE_ISO
- C7 pad 1: VCC_ISO -> Net-(C7-Pad1)
- C7 pad 2: VEE_ISO -> GND_ISO
- C8 pad 2: GND_ISO -> VEE_ISO
- C9 pad 1: GND_ISO -> VCC_ISO
- C9 pad 2: VEE_ISO -> GND_ISO
- R6 pad 2: Net-(C6-Pad1) -> Net-(C7-Pad1)
- U1 pad 15: Net-(C6-Pad1) -> Net-(C7-Pad1)
Routing:
- net VEE_ISO: track 0.00 -> 105.8 mm
- net GND_ISO: track 0.00 -> 96.1 mm, vias 0 -> 4
- net +15V: track 0.00 -> 76.5 mm
- net VCC_ISO: track 0.00 -> 75.1 mm, vias 0 -> 4
- net VCC: track 0.00 -> 65.4 mm, vias 0 -> 2
- net GND: track 0.00 -> 65.1 mm, vias 0 -> 2
- net Net-(J4-Pad2): track 0.00 -> 63.8 mm, vias 0 -> 1
- net Net-(D2-Pad1): track 0.00 -> 38.2 mm
- net Net-(J1-Pad3): track 0.00 -> 29.2 mm
- net Net-(J1-Pad4): track 0.00 -> 28.7 mm
- net Net-(J1-Pad5): track 0.00 -> 28.2 mm
- net Net-(J1-Pad6): track 0.00 -> 27.6 mm
- net Net-(J1-Pad7): track 0.00 -> 27.1 mm
- net Net-(R5-Pad2): track 0.00 -> 24.9 mm, vias 0 -> 1
- net Net-(R4-Pad2): track 0.00 -> 24.1 mm, vias 0 -> 1
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- added copper zone on B.Cu, net GND
- added copper zone on B.Cu, net GND_ISO
Other:
- net class Default: trace_width 0.25 -> 1.5; via_dia 0.6 -> 1; via_drill 0.4 -> 0.5

Commit message: Minor layout changes
Parts:
- added REF**: MountingHole_4.3mm_M4_ISO7380_Pad, Mounting_Holes:MountingHole_4.3mm_M4_ISO7380_Pad, F.Cu at (187.2, 150.7)
- added REF**: MountingHole_4.3mm_M4_ISO7380_Pad, Mounting_Holes:MountingHole_4.3mm_M4_ISO7380_Pad, F.Cu at (187.5, 119.0)
- added REF**: MountingHole_4.3mm_M4_ISO7380_Pad, Mounting_Holes:MountingHole_4.3mm_M4_ISO7380_Pad, F.Cu at (93.0, 116.8)
- added REF**: MountingHole_4.3mm_M4_ISO7380_Pad, Mounting_Holes:MountingHole_4.3mm_M4_ISO7380_Pad, F.Cu at (94.0, 152.0)
- moved TP1 8.36 mm to (167.6, 116.6)
- moved D2 7.58 mm to (174.7, 116.7)
Routing:
- net Net-(D2-Pad1): track 38.2 -> 47.4 mm
- net Net-(D2-Pad2): track 4.29 -> 11.8 mm
- net VEE_ISO: track 105.8 -> 102.1 mm
- net GND_ISO: track 96.1 -> 93.4 mm
- net Net-(D4-Pad2): track 8.16 -> 6.65 mm
Other:
- board outline added: 90.6 x 41.8 mm
- board text added: "Don't blame me. I'm an interpreter. I'm not supposed to know a power socket from a computer terminal."
