File: Flyback2000/Flyback2000.sch (KiCad schematic (older format))
At the start: 54 parts, among them Q1 BC413C, Q2 BC413C, Q3 Q_PNP_BCE, Q4 2N7002, T1 Transformer_2P_3S, U1 OPA2333D, U2 OPTO-TRANSISTOR-4

Commit message: Added Texas controller to schematic. Correct symbol ?
Parts:
- added U?: LM2587, symbol LM2587
Changed lines of the file:
@@
 LIBS:contrib
 LIBS:valves
+LIBS:Flyback2000-cache
 EELAYER 25 0
 EELAYER END
@@
 Wire Wire Line
 	4600 6800 4600 6700
+$Comp
+L LM2587 U?
+U 1 1 5986E761
+P 2950 3050
+F 0 "U?" H 2600 3300 60  0000 C CNN
+F 1 "LM2587" H 2950 3100 60  0000 C CNN
+F 2 "" H 2950 3050 60  0001 C CNN
+F 3 "" H 2950 3050 60  0001 C CNN
+	1    2950 3050
+	1    0    0    -1
+$EndComp
 $EndSCHEMATC

Commit message: The LM2587 has a different purpose
Parts:
- removed U?: LM2587, symbol LM2587
- added U?: TL494, symbol TL494
Changed lines of the file:
@@
 LIBS:contrib
 LIBS:valves
+LIBS:Texas
 LIBS:Flyback2000-cache
 EELAYER 25 0
@@
 	4600 6800 4600 6700
 $Comp
-L LM2587 U?
-U 1 1 5986E761
-P 2950 3050
-F 0 "U?" H 2600 3300 60  0000 C CNN
-F 1 "LM2587" H 2950 3100 60  0000 C CNN
-F 2 "" H 2950 3050 60  0001 C CNN
-F 3 "" H 2950 3050 60  0001 C CNN
-	1    2950 3050
-	1    0    0    -1
-$EndComp
+L TL494 U?
+U 1 1 59875519
+P 2900 2950
+F 0 "U?" H 2600 3600 60  0000 C CNN
+F 1 "TL494" H 2700 2250 60  0000 C CNN
+F 2 "" H 2900 2900 60  0001 C CNN
+F 3 "" H 2900 2900 60  0001 C CNN
+	1    2900 2950
+	1    0    0    -1
+$EndComp

Commit message: Updated components
Parts:
- removed D10: Q_Thyristor_AGK, symbol Q_Thyristor_AGK
- removed U?: TL494, symbol TL494
- added D?: TL431LP, TO_SOT_Packages_THT:TO-92_Inline_Narrow_Oval, symbol TL431LP
- added U?: TL494, symbol TL494
Connections:
- wire segments 138 -> 156
- no-connect marks 0 -> 2
Other:
- moved on the sheet: R5

Commit message: improved readability of schematic
Parts:
- added U4: LM7815ACT, TO_SOT_Packages_THT:TO-220_Vertical, symbol LM7815ACT
- added U5: LM7915CT, TO_SOT_Packages_THT:TO-220_Vertical, symbol LM7915CT
- gave numbers to parts that had none: 2
Connections:
- wire segments 156 -> 146
Other:
- moved on the sheet: C1, C2, R1, R2, R3

Commit message: Redrawn schematic, added component values and ratings, changed diodes to correct type
Parts:
- removed D1: D_Bridge_+-AA, symbol D_Bridge_+-AA
- removed D5, D6: D, symbol D
- removed U1: OPA2333D, symbol OPA2333D
- added D?: 1N4148, Diodes_THT:D_DO-35_SOD27_Horizontal_RM10, symbol 1N4148
- added D? (x5): 1N4007, Diodes_THT:D_DO-41_SOD81_Horizontal_RM10, symbol 1N4007
- added U?: LM393, symbol LM393
- C10, C13, C14, C9: value C -> 100u
- C11, C15: value C -> 330u
- C5, C7: value CP -> 100u
- C6: value C -> 22u
- D2: value D_Zener -> 15V
- F1: value Fuse -> 1A
- R1: value R -> 5k
- R10, R11, R9: value R -> 10k; Power Rating (none) -> 2W
- R13: Power Rating (none) -> 2W
- R14: value R -> 0.1; Power Rating (none) -> 2W
- R2: value R_Variable -> 10k
- R4: value R -> 1k
Connections:
- net labels removed: VCC
- wire segments 146 -> 152
Other:
- moved on the sheet: C1, C10, C11, C12, C13, C14, C15, C2, C3, C4, C5, C6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

Commit message: More layout changes and annotation/footprint assosiations
Parts:
- removed D7, D8, D9: D, symbol D
- added D10, D11, D12: 1N4148, Diodes_THT:D_DO-35_SOD27_Horizontal_RM10, symbol 1N4148
- added J1: CONN_01X03, symbol CONN_01X03
- added J2, J3, J4: CONN_01X02, symbol CONN_01X02
- C1, C2: footprint (none) -> Capacitors_SMD:C_1206_HandSoldering
- C5: footprint (none) -> Capacitors_SMD:CP_Elec_6.3x7.7
- C6: renamed from C7; footprint (none) -> Capacitors_SMD:CP_Elec_6.3x7.7
- D6: renamed from D4; value D_Zener -> 15V
- F1: footprint (none) -> Fuse_Holders_and_Fuses:Fuseholder5x20_vert_closed_Bulgin_FX0456
- R1, R3: footprint (none) -> Resistors_SMD:R_1206_HandSoldering
- R4: renamed from R5; footprint (none) -> Resistors_SMD:R_1206_HandSoldering
- R7: renamed from R4; footprint (none) -> Resistors_SMD:R_1206_HandSoldering
- RV1: value Varistor -> MOV
- gave numbers to parts that had none: 7
- renumbered C9 to C10, C10 to C11, C11 to C12, C6 to C7, C12 to C9, D10 to D13, D3 to D5, D2 to D7, R11 to R10, R13 to R11, R6 to R12, R7 to R13, R18 to R15, R15 to R16, R16 to R17, R17 to R18, R8 to R5, R12 to R6, R9 to R8, R10 to R9, U3 to U1, U2 to U3
Connections:
- net labels removed: +15V, +5V, AC
- wire segments 152 -> 166
Other:
- moved on the sheet: F1, Q1

Commit message: Minor change to .gitignore, and upload of some new projects
Parts:
- R18: value R -> 1k
Changed lines of the file:
@@
 LIBS:graphic
 LIBS:hc11
-LIBS:intersil
 LIBS:ir
 LIBS:Lattice
@@
 LIBS:Zilog
 LIBS:custom_transformers
-LIBS:Flyback2000-cache
 EELAYER 25 0
 EELAYER END
@@
 P 8250 3500
 F 0 "R18" V 8330 3500 50  0000 C CNN
-F 1 "R" V 8250 3500 50  0000 C CNN
+F 1 "1k" V 8250 3500 50  0000 C CNN
 F 2 "" V 8180 3500 50  0001 C CNN
 F 3 "" H 8250 3500 50  0001 C CNN
