File: Current_Sensor/Current_sensor.sch (KiCad schematic (older format))
At the start: 38 parts, among them P1 CONN_01X04, P2 CONN_01X02, P3 CONN_01X03, U1 LTS-25-NP, U2 LTS-25-NP, U3 LTS-25-NP, U4 NE5532, U5 NE5532, U6 NE5532

Commit message: Updated current sensor card
Parts:
- added D3: LED, LEDs:LED_1206_HandSoldering, symbol LED
- added R18: R, Resistors_SMD:R_1206_HandSoldering, symbol R
- C6, C7: footprint Capacitors_ThroughHole:C_Radial_D22_L41_P10 -> Capacitors_THT:CP_Radial_D5.0mm_P2.50mm
- D1, D2: footprint LEDs:LED_1206 -> LEDs:LED_1206_HandSoldering
- RV1, RV2, RV3: footprint potentiometer:Potentiometer_Trimmer-Suntan-TSR-3386P -> Potentiometers:Potentiometer_Trimmer_ACP_CA6v_Horizontal
Connections:
- wire segments 78 -> 81
Other:
- moved on the sheet: D2, R17, RV1, RV2, RV3

Commit message: Corrected library reference to phoenix connectors
Parts:
- P1: footprint phoenix:PhoenixContact_MSTBA-G_04x5.00mm_Angled -> PhoenixContact:MSTBA_25_4p_G_508-1757268
- P2: footprint phoenix:PhoenixContact_MSTBA-G_02x5.00mm_Angled -> PhoenixContact:MSTBA_25_2p_G_508-1757242
- P3: footprint phoenix:PhoenixContact_MSTBA-G_03x5.00mm_Angled -> PhoenixContact:MSTBA_25_3p_G_508-1757488
Changed lines of the file:
@@
 F 0 "P2" H 8150 5800 50  0000 C CNN
 F 1 "CONN_01X02" V 8250 5650 50  0000 C CNN
-F 2 "phoenix:PhoenixContact_MSTBA-G_02x5.00mm_Angled" H 8150 5650 50  0001 C CNN
+F 2 "PhoenixContact:MSTBA_25_2p_G_508-1757242" H 8150 5650 50  0001 C CNN
 F 3 "" H 8150 5650 50  0000 C CNN
 	1    8150 5650
@@
 F 0 "P3" H 8150 6450 50  0000 C CNN
 F 1 "CONN_01X03" V 8250 6250 50  0000 C CNN
-F 2 "phoenix:PhoenixContact_MSTBA-G_03x5.00mm_Angled" H 8150 6250 50  0001 C CNN
+F 2 "PhoenixContact:MSTBA_25_3p_G_508-1757488" H 8150 6250 50  0001 C CNN
 F 3 "" H 8150 6250 50  0000 C CNN
 	1    8150 6250
@@
 F 0 "P1" H 7600 4000 50  0000 C CNN
 F 1 "CONN_01X04" V 7700 3750 50  0000 C CNN
-F 2 "phoenix:PhoenixContact_MSTBA-G_04x5.00mm_Angled" H 7600 3750 50  0001 C CNN
+F 2 "PhoenixContact:MSTBA_25_4p_G_508-1757268" H 7600 3750 50  0001 C CNN
 F 3 "" H 7600 3750 50  0000 C CNN
 	1    7600 3750

Commit message: Added component values for bias adjustment
Parts:
- C1, C2, C3: value C -> 100n
- R4, R6, R7, R8, R9: value R -> 10k
- RV1, RV2, RV3: value POT -> 10k
Changed lines of the file:
@@
 U 1 1 583F1C1C
 P 3800 3600
-F 0 "RV2" H 3800 3520 50  0000 C CNN
-F 1 "POT" H 3800 3600 50  0000 C CNN
+F 0 "RV2" V 3700 3600 50  0000 C CNN
+F 1 "10k" V 3800 3600 50  0000 C CNN
 F 2 "Potentiometers:Potentiometer_Trimmer_ACP_CA6v_Horizontal" H 3800 3600 50  0001 C CNN
 F 3 "" H 3800 3600 50  0000 C CNN
@@
 U 1 1 583F1C94
 P 3800 3200
-F 0 "R6" V 3880 3200 50  0000 C CNN
-F 1 "R" V 3800 3200 50  0000 C CNN
+F 0 "R6" V 3700 3200 50  0000 C CNN
+F 1 "10k" V 3800 3200 50  0000 C CNN
 F 2 "Resistors_SMD:R_1206_HandSoldering" V 3730 3200 50  0001 C CNN
 F 3 "" H 3800 3200 50  0000 C CNN
@@
 U 1 1 583F1CDF
 P 3800 4100
-F 0 "R7" V 3880 4100 50  0000 C CNN
-F 1 "R" V 3800 4100 50  0000 C CNN
+F 0 "R7" V 3700 4100 50  0000 C CNN
+F 1 "10k" V 3800 4100 50  0000 C CNN
 F 2 "Resistors_SMD:R_1206_HandSoldering" V 3730 4100 50  0001 C CNN
 F 3 "" H 3800 4100 50  0000 C CNN
@@
 U 1 1 58453742
 P 3800 1450
-F 0 "RV1" H 3800 1370 50  0000 C CNN
-F 1 "POT" H 3800 1450 50  0000 C CNN
+F 0 "RV1" V 3700 1450 50  0000 C CNN
+F 1 "10k" V 3800 1450 50  0000 C CNN
 F 2 "Potentiometers:Potentiometer_Trimmer_ACP_CA6v_Horizontal" H 3800 1450 50  0001 C CNN
 F 3 "" H 3800 1450 50  0000 C CNN
@@
 U 1 1 58453748
 P 3800 1050
-F 0 "R4" V 3880 1050 50  0000 C CNN
-F 1 "R" V 3800 1050 50  0000 C CNN
+F 0 "R4" V 3700 1050 50  0000 C CNN
+F 1 "10k" V 3800 1050 50  0000 C CNN
 F 2 "Resistors_SMD:R_1206_HandSoldering" V 3730 1050 50  0001 C CNN
 F 3 "" H 3800 1050 50  0000 C CNN
@@
 U 1 1 5845374E
 P 3800 1950
-F 0 "R5" V 3880 1950 50  0000 C CNN
+F 0 "R5" V 3700 1950 50  0000 C CNN
 F 1 "R" V 3800 1950 50  0000 C CNN
 F 2 "Resistors_SMD:R_1206_HandSoldering" V 3730 1950 50  0001 C CNN
@@
 P 5200 1150
 F 0 "C1" H 5225 1250 50  0000 L CNN
-F 1 "C" H 5225 1050 50  0000 L CNN
+F 1 "100n" H 5225 1050 50  0000 L CNN
 F 2 "Capacitors_SMD:C_1206_HandSoldering" H 5238 1000 50  0001 C CNN
 F 3 "" H 5200 1150 50  0000 C CNN
@@
 U 1 1 58453A12
 P 3800 5750
-F 0 "RV3" H 3800 5670 50  0000 C CNN
-F 1 "POT" H 3800 5750 50  0000 C CNN
+F 0 "RV3" V 3700 5750 50  0000 C CNN
+F 1 "10k" V 3800 5750 50  0000 C CNN
 F 2 "Potentiometers:Potentiometer_Trimmer_ACP_CA6v_Horizontal" H 3800 5750 50  0001 C CNN
 F 3 "" H 3800 5750 50  0000 C CNN
@@
 U 1 1 58453A18
 P 3800 5350
-F 0 "R8" V 3880 5350 50  0000 C CNN
-F 1 "R" V 3800 5350 50  0000 C CNN
+F 0 "R8" V 3700 5350 50  0000 C CNN
+F 1 "10k" V 3800 5350 50  0000 C CNN
 F 2 "Resistors_SMD:R_1206_HandSoldering" V 3730 5350 50  0001 C CNN
 F 3 "" H 3800 5350 50  0000 C CNN
@@
 U 1 1 58453A1E
 P 3800 6250
-F 0 "R9" V 3880 6250 50  0000 C CNN
-F 1 "R" V 3800 6250 50  0000 C CNN
+F 0 "R9" V 3700 6250 50  0000 C CNN
+F 1 "10k" V 3800 6250 50  0000 C CNN
 F 2 "Resistors_SMD:R_1206_HandSoldering" V 3730 6250 50  0001 C CNN
 F 3 "" H 3800 6250 50  0000 C CNN
@@
 P 5200 5450
 F 0 "C3" H 5225 5550 50  0000 L CNN
-F 1 "C" H 5225 5350 50  0000 L CNN
+F 1 "100n" H 5225 5350 50  0000 L CNN
 F 2 "Capacitors_SMD:C_1206_HandSoldering" H 5238 5300 50  0001 C CNN
 F 3 "" H 5200 5450 50  0000 C CNN
@@
 P 5200 3250
 F 0 "C2" H 5225 3350 50  0000 L CNN
-F 1 "C" H 5225 3150 50  0000 L CNN
+F 1 "100n" H 5225 3150 50  0000 L CNN
 F 2 "Capacitors_SMD:C_1206_HandSoldering" H 5238 3100 50  0001 C CNN
 F 3 "" H 5200 3250 50  0000 C CNN

Commit message: Added component values as soldered
Parts:
- R17: value R -> 250
- R5: value R -> 10k
Changed lines of the file:
@@
 P 3800 1950
 F 0 "R5" V 3700 1950 50  0000 C CNN
-F 1 "R" V 3800 1950 50  0000 C CNN
+F 1 "10k" V 3800 1950 50  0000 C CNN
 F 2 "Resistors_SMD:R_1206_HandSoldering" V 3730 1950 50  0001 C CNN
 F 3 "" H 3800 1950 50  0000 C CNN
@@
 P 10400 4200
 F 0 "R17" V 10480 4200 50  0000 C CNN
-F 1 "R" V 10400 4200 50  0000 C CNN
+F 1 "250" V 10400 4200 50  0000 C CNN
 F 2 "Resistors_SMD:R_1206_HandSoldering" V 10330 4200 50  0001 C CNN
 F 3 "" H 10400 4200 50  0000 C CNN

Commit message: Updated component values and highlighted errors and/or improvement possibilities for next revision
Parts:
- C4, C5: value C -> 100n
- C6, C7: value CP -> 47u
- D1: value LED -> RED
- D2: value LED -> GREEN; Color (none) -> Green
- R1: value R -> 1k
- R10: value R -> 0R
- R13: value R -> open
- R16, R18: value R -> 2k
- renumbered D3 to YELLOW
Connections:
- wire segments 81 -> 85
Other:
- note added: "Next rev: Potmeter here..."
- moved on the sheet: C4, C5, C6, C7
Changed lines of the file:
@@
 L CP C6
 U 1 1 584407EF
-P 9900 5950
-F 0 "C6" H 9925 6050 50  0000 L CNN
-F 1 "CP" H 9925 5850 50  0000 L CNN
-F 2 "Capacitors_THT:CP_Radial_D5.0mm_P2.50mm" H 9938 5800 50  0001 C CNN
-F 3 "" H 9900 5950 50  0000 C CNN
-	1    9900 5950
+P 9900 6000
+F 0 "C6" H 9925 6100 50  0000 L CNN
+F 1 "47u" H 9925 5900 50  0000 L CNN
+F 2 "Capacitors_THT:CP_Radial_D5.0mm_P2.50mm" H 9938 5850 50  0001 C CNN
+F 3 "" H 9900 6000 50  0000 C CNN
+	1    9900 6000
 	1    0    0    -1
 $EndComp
@@
 L CP C7
 U 1 1 58440842
-P 9900 6550
-F 0 "C7" H 9925 6650 50  0000 L CNN
-F 1 "CP" H 9925 6450 50  0000 L CNN
-F 2 "Capacitors_THT:CP_Radial_D5.0mm_P2.50mm" H 9938 6400 50  0001 C CNN
-F 3 "" H 9900 6550 50  0000 C CNN
-	1    9900 6550
+P 9900 6500
+F 0 "C7" H 9925 6600 50  0000 L CNN
+F 1 "47u" H 9925 6400 50  0000 L CNN
+F 2 "Capacitors_THT:CP_Radial_D5.0mm_P2.50mm" H 9938 6350 50  0001 C CNN
+F 3 "" H 9900 6500 50  0000 C CNN
+	1    9900 6500
 	1    0    0    -1
 $EndComp
@@
 L C C4
 U 1 1 58440C87
-P 9550 5950
-F 0 "C4" H 9575 6050 50  0000 L CNN
-F 1 "C" H 9575 5850 50  0000 L CNN
-F 2 "Capacitors_SMD:C_1206_HandSoldering" H 9588 5800 50  0001 C CNN
-F 3 "" H 9550 5950 50  0000 C CNN
-	1    9550 5950
+P 9550 6000
+F 0 "C4" H 9575 6100 50  0000 L CNN
+F 1 "100n" H 9575 5900 50  0000 L CNN
+F 2 "Capacitors_SMD:C_1206_HandSoldering" H 9588 5850 50  0001 C CNN
+F 3 "" H 9550 6000 50  0000 C CNN
+	1    9550 6000
 	1    0    0    -1
 $EndComp
@@
 L C C5
 U 1 1 58440CFB
-P 9550 6550
-F 0 "C5" H 9575 6650 50  0000 L CNN
-F 1 "C" H 9575 6450 50  0000 L CNN
-F 2 "Capacitors_SMD:C_1206_HandSoldering" H 9588 6400 50  0001 C CNN
-F 3 "" H 9550 6550 50  0000 C CNN
-	1    9550 6550
+P 9550 6500
+F 0 "C5" H 9575 6600 50  0000 L CNN
+F 1 "100n" H 9575 6400 50  0000 L CNN
+F 2 "Capacitors_SMD:C_1206_HandSoldering" H 9588 6350 50  0001 C CNN
+F 3 "" H 9550 6500 50  0000 C CNN
+	1    9550 6500
 	1    0    0    -1
 $EndComp
@@
 	8950 6150 8350 6150
 Wire Wire Line
-	9550 6100 9550 6400
-Wire Wire Line
-	9900 6100 9900 6400
-Wire Wire Line
 	8350 6250 10800 6250
 Connection ~ 9900 6250
@@
 P 2950 1650
 F 0 "R1" V 3030 1650 50  0000 C CNN
-F 1 "R" V 2950 1650 50  0000 C CNN
+F 1 "1k" V 2950 1650 50  0000 C CNN
 F 2 "Resistors_SMD:R_1206_HandSoldering" V 2880 1650 50  0001 C CNN
 F 3 "" H 2950 1650 50  0000 C CNN
@@
 P 5800 1550
 F 0 "R10" V 5880 1550 50  0000 C CNN
-F 1 "R" V 5800 1550 50  0000 C CNN
+F 1 "0R" V 5800 1550 50  0000 C CNN
 F 2 "Resistors_SMD:R_1206_HandSoldering" V 5730 1550 50  0001 C CNN
 F 3 "" H 5800 1550 50  0000 C CNN
@@
 P 6050 1950
 F 0 "R13" V 6130 1950 50  0000 C CNN
-F 1 "R" V 6050 1950 50  0000 C CNN
+F 1 "open" V 6050 1950 50  0000 C CNN
 F 2 "Resistors_SMD:R_1206_HandSoldering" V 5980 1950 50  0001 C CNN
 F 3 "" H 6050 1950 50  0000 C CNN
@@
 P 9950 3750
 F 0 "D1" H 9950 3850 50  0000 C CNN
-F 1 "LED" H 9950 3650 50  0000 C CNN
+F 1 "RED" H 9950 3650 50  0000 C CNN
 F 2 "LEDs:LED_1206_HandSoldering" H 9950 3750 50  0001 C CNN
 F 3 "" H 9950 3750 50  0000 C CNN
@@
 P 10400 3750
 F 0 "D2" H 10400 3850 50  0000 C CNN
-F 1 "LED" H 10400 3650 50  0000 C CNN
+F 1 "GREEN" H 10400 3650 50  0000 C CNN
 F 2 "LEDs:LED_1206_HandSoldering" H 10400 3750 50  0001 C CNN
 F 3 "" H 10400 3750 50  0000 C CNN
+F 4 "Green" H 10400 3750 60  0001 C CNN "Color"
 	1    10400 3750
 	0    -1   -1   0
@@
 P 9950 4200
 F 0 "R16" V 10030 4200 50  0000 C CNN
-F 1 "R" V 9950 4200 50  0000 C CNN
+F 1 "2k" V 9950 4200 50  0000 C CNN
 F 2 "Resistors_SMD:R_1206_HandSoldering" V 9880 4200 50  0001 C CNN
 F 3 "" H 9950 4200 50  0000 C CNN
@@
 LEDs for power supply
 $Comp
-L LED D3
+L LED YELLOW
 U 1 1 5981D266
 P 10850 3750
-F 0 "D3" H 10850 3850 50  0000 C CNN
+F 0 "YELLOW" H 10850 3850 50  0000 C CNN
 F 1 "LED" H 10850 3650 50  0000 C CNN
 F 2 "LEDs:LED_1206_HandSoldering" H 10850 3750 50  0001 C CNN
@@
 P 10850 4200
 F 0 "R18" V 10930 4200 50  0000 C CNN
-F 1 "R" V 10850 4200 50  0000 C CNN
+F 1 "2k" V 10850 4200 50  0000 C CNN
 F 2 "Resistors_SMD:R_1206_HandSoldering" V 10780 4200 50  0001 C CNN
 F 3 "" H 10850 4200 50  0000 C CNN
@@
 	-1   0    0    -1
 $EndComp
+Text Notes 4250 4400 0    60   ~ 0
+Next rev: Potmeter here...
+Wire Wire Line
+	9900 5800 9900 5850
+Wire Wire Line
+	9550 5850 9550 5800
+Wire Wire Line
+	9550 6150 9550 6350
+Wire Wire Line
+	9900 6150 9900 6350
+Wire Wire Line
+	9900 6700 9900 6650
+Wire Wire Line
+	9550 6650 9550 6700
 $EndSCHEMATC

Commit message: Removed hard-coded paths
Parts:
- C1, C2, C3, C4, C5: symbol C -> device:C
- C6, C7: symbol CP -> device:CP
- D1, D2, YELLOW: symbol LED -> device:LED
- P1: symbol CONN_01X04 -> conn:Conn_01x04
- P2: symbol CONN_01X02 -> conn:Conn_01x02
- P3: symbol CONN_01X03 -> conn:Conn_01x03
- R1, R10, R11, R12, R13, R14, R15, R16, R17, R18, R2, R3, R4, R5, R6, R7, R8, R9: symbol R -> device:R
- RV1, RV2, RV3: symbol POT -> device:POT
- U1, U2, U3: symbol LTS-25-NP -> LEM:LTS-25-NP
- U4, U5, U6: symbol NE5532 -> linear:NE5532
Connections:
- wire segments 85 -> 100
