File: Inverter_card_2/Inverter_card_2.kicad_pcb (KiCad board)
At the start: 2 copper layers, 34 parts, among them J1 CONN_01X01, J2 CONN_01X01, J3 CONN_01X01, P1 CONN_01X03, P10 CONN_01X02, P15 CONN_01X03, P16 CONN_01X03, P2 CONN_01X03, P20 CONN_01X02, P22 CONN_01X02, P3 CONN_01X03, P4 CONN_01X03, P5 CONN_01X03, P6 CONN_01X03, T1 SemikronSKiiP_13ACM12V18, U1 LTS-25-NP, U2 LTS-25-NP, U3 LTS-25-NP

Commit message: Created netlist and spread out footprints on .kicad-pcb file.
Parts:
- removed D1: GREEN, LEDs:LED_1206_HandSoldering
- removed J1, J2, J3: CONN_01X01, Pin_Headers:Pin_Header_Straight_1x01_Pitch2.54mm
- removed P10, P22: CONN_01X02, PhoenixContact:MSTBA_25_2p_G_508-1757242
- removed P15, P16: CONN_01X03, PhoenixContact:MSTBA_25_3p_G_508-1757488
- removed U1, U2, U3: LTS-25-NP, LEM:LTS25-NP
- added C15: 100nF, Capacitors_SMD:C_1206_HandSoldering, F.Cu at (446.6, 179.6)
- added C16: 100nF, Capacitors_SMD:C_1206_HandSoldering, F.Cu at (482.2, 143.5)
- added C22: 10nF, Capacitors_SMD:C_1206_HandSoldering, F.Cu at (446.6, 185.4)
- added C31: 10uF, Capacitors_SMD:C_1210_HandSoldering, F.Cu at (489.2, 141.7)
- added C41: 100pF, Capacitors_SMD:C_1210_HandSoldering, F.Cu at (453.5, 180.1)
- added C42: 100nF, Capacitors_SMD:C_1210_HandSoldering, F.Cu at (465.1, 172.7)
- added C43: 100nF, Capacitors_SMD:C_1206_HandSoldering, F.Cu at (433.5, 214.9)
- added C51: 100pF, Capacitors_SMD:C_1210_HandSoldering, F.Cu at (476.6, 162.3)
- added C52: 100nF, Capacitors_SMD:C_1210_HandSoldering, F.Cu at (496.1, 141.7)
- added C53: 100nF, Capacitors_SMD:C_1206_HandSoldering, F.Cu at (460.5, 184.8)
- added CP21: 10uF, Capacitors_SMD:CP_Elec_6.3x7.7, F.Cu at (472.1, 153.6)
- added D21: GREEN, LEDs:LED_1206_HandSoldering, F.Cu at (425.7, 215.9)
- added D31: GREEN, LEDs:LED_1206_HandSoldering, F.Cu at (446.6, 191.3)
- added P0: CONN_01X03, PhoenixContact:MSTBA_25_3p_G_508-1757488, F.Cu at (471.4, 111.4)
- added P7: CONN_01X03, PhoenixContact:MSTBA_25_3p_G_508-1757488, F.Cu at (387.5, 203.2)
- added R11: 250, Resistors_SMD:R_1206_HandSoldering, F.Cu at (503.1, 141.3)
- added R12: 250, Resistors_SMD:R_1206_HandSoldering, F.Cu at (497.1, 148.1)
- added R13: 250, Resistors_SMD:R_1206_HandSoldering, F.Cu at (472.0, 168.7)
- added R21: 1250, Resistors_SMD:R_1206_HandSoldering, F.Cu at (446.6, 197.1)
- added R31: 1250, Resistors_SMD:R_1206_HandSoldering, F.Cu at (490.2, 153.9)
- added R41: 100k, Resistors_THT:R_Axial_DIN0414_L11.9mm_D4.5mm_P15.24mm_Horizontal, F.Cu at (385.0, 194.6)
- added R5: 100k, Resistors_SMD:R_1206_HandSoldering, F.Cu at (460.5, 179.1)
- added R51: 2.7M, Resistors_SMD:R_2010_HandSoldering, F.Cu at (481.9, 151.4)
- added R52: 2.7M, Resistors_SMD:R_2010_HandSoldering, F.Cu at (425.2, 209.6)
- added R53: 20k, Resistors_SMD:R_1206_HandSoldering, F.Cu at (490.2, 148.1)
- added R6: 100k, Resistors_SMD:R_1206_HandSoldering, F.Cu at (483.6, 159.7)
- added R8: 200k, Resistors_SMD:R_2512_HandSoldering, F.Cu at (473.0, 144.3)
- added R9: 200k, Resistors_SMD:R_2512_HandSoldering, F.Cu at (448.9, 173.1)
- added TP1: TEST, Measurement_Points:Test_Point, F.Cu at (495.1, 154.0)
- added TP10: TEST, Measurement_Points:Test_Point, F.Cu at (451.5, 198.5)
- added TP11: TEST, Measurement_Points:Test_Point, F.Cu at (465.4, 180.4)
- added TP12: TEST, Measurement_Points:Test_Point, F.Cu at (470.9, 180.4)
- added TP2: TEST, Measurement_Points:Test_Point, F.Cu at (444.6, 203.1)
- added TP21: TEST, Measurement_Points:Test_Point, F.Cu at (465.4, 186.5)
- added TP22: TEST, Measurement_Points:Test_Point, F.Cu at (483.9, 165.9)
- added TP3: TEST, Measurement_Points:Test_Point, F.Cu at (438.4, 209.4)
- added TP31: TEST, Measurement_Points:Test_Point, F.Cu at (443.8, 209.4)
- added TP32: TEST, Measurement_Points:Test_Point, F.Cu at (477.0, 174.6)
- added TP4: TEST, Measurement_Points:Test_Point, F.Cu at (451.5, 192.5)
- added TP5: TEST, Measurement_Points:Test_Point, F.Cu at (501.6, 133.9)
- added TP6: TEST, Measurement_Points:Test_Point, F.Cu at (379.0, 213.5)
- added TP7: TEST, Measurement_Points:Test_Point, F.Cu at (488.5, 159.8)
- added TP8: TEST, Measurement_Points:Test_Point, F.Cu at (502.1, 147.2)
- added TP9: TEST, Measurement_Points:Test_Point, F.Cu at (457.0, 192.5)
- added U11: ACS758xCB-PFF, Allegro:ACS758LCB-050B-PFF-T, F.Cu at (354.0, 216.8)
- added U12: ACS758xCB-PFF, Allegro:ACS758LCB-050B-PFF-T, F.Cu at (334.1, 216.8)
- added U13: ACS758xCB-PFF, Allegro:ACS758LCB-050B-PFF-T, F.Cu at (314.2, 216.8)
- added U30: ISE0505A-H, Housings_DIP:DIP-8_W11.48mm_SMD, F.Cu at (492.9, 131.2)
- added U40: ACPL-C87B, Housings_SOIC:SSO-8_6.8x5.9mm_Pitch1.27mm_Clearance8mm, F.Cu at (370.7, 215.4)
- added U50: ACPL-C87B, Housings_SOIC:SSO-8_6.8x5.9mm_Pitch1.27mm_Clearance8mm, F.Cu at (408.5, 212.0)
- C1, C2, C3, C4: value C -> 50uF
- C11, C12: value CP -> 100nF; footprint Capacitors_SMD:CP_Elec_6.3x7.7 -> Capacitors_SMD:C_1206_HandSoldering
- C13, C14: value C -> 100nF
- C5, C6: footprint Capacitors_THT:C_Rect_L16.5mm_W8.7mm_P15.00mm_MKT -> Capacitors_THT:C_Rect_L19.0mm_W5.0mm_P15.00mm_MKS4
- C7: value C -> 22pF; footprint Capacitors_THT:C_Rect_L16.5mm_W8.7mm_P15.00mm_MKT -> Capacitors_THT:C_Rect_L19.0mm_W5.0mm_P15.00mm_MKS4
- R1, R2, R3: value R -> 100k; footprint Resistors_THT:R_Axial_DIN0414_L11.9mm_D4.5mm_P15.24mm_Horizontal -> Resistors_SMD:R_1206_HandSoldering
- R4: value 250 -> 100k
- T1: value SemikronSKiiP_13ACM12V18 -> SKiiP_13ACM12V18
- moved P4 389.1 mm to (481.4, 136.5)
- moved P3 373.0 mm to (416.1, 202.8)
- moved R3 370.9 mm to (502.9, 127.5)
- moved P1 368.6 mm to (428.9, 193.8)
- moved T1 362.1 mm to (445.9, 127.5)
- moved P2 347.5 mm to (438.5, 156.9)
- moved R2 340.3 mm to (453.5, 186.6)
- moved P5 337.5 mm to (489.9, 111.4)
- moved R1 335.2 mm to (418.8, 215.9)
- moved C12 317.5 mm to (458.1, 172.2)
- moved C7 313.1 mm to (429.4, 155.3)
- moved C14 312.1 mm to (479.0, 168.8)
- moved C11 311.2 mm to (469.7, 161.8)
- moved C13 308.1 mm to (472.0, 174.6)
- moved C5 284.2 mm to (368.7, 192.9)
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Connections:
- C11 pad 1: Net-(C11-Pad1) -> VCC
- C11 pad 2: Net-(C11-Pad2) -> GND
- C12 pad 1: Net-(C11-Pad2) -> VCC
- C12 pad 2: Net-(C12-Pad2) -> GND
- C13 pad 1: Net-(C11-Pad1) -> VCC
- C13 pad 2: Net-(C13-Pad2) -> GND
- C14 pad 1: Net-(C13-Pad2) -> Net-(C14-Pad1)
- C14 pad 2: Net-(C12-Pad2) -> GND
- C2 pad 2: DC- -> GND_ISO
- C4 pad 2: DC- -> GND_ISO
- C5 pad 2: Net-(C5-Pad2) -> Net-(C1-Pad2)
- C6 pad 1: Net-(C5-Pad2) -> Net-(C1-Pad2)
- C6 pad 2: DC- -> GND_ISO
- C7 pad 2: Net-(C7-Pad2) -> (no net)
- P2 pad 3: DC- -> GND_ISO
- P20 pad 1: Net-(C11-Pad1) -> VCC
- P20 pad 2: Net-(C12-Pad2) -> GND
- P4 pad 2: T5_g -> T4_g
- P4 pad 3: DC- -> GND_ISO
- P5 pad 2: T4_g -> T5_g
- P6 pad 3: DC- -> GND_ISO
- R1 pad 1: DC+ -> T1_g
- R1 pad 2: Net-(C1-Pad2) -> U
- R2 pad 1: Net-(C1-Pad2) -> T2_g
- R2 pad 2: DC- -> GND_ISO
- R3 pad 1: Net-(C7-Pad2) -> T3_g
- R3 pad 2: DC- -> V
- R4 pad 1: Net-(C11-Pad1) -> T4_g
- R4 pad 2: Net-(D1-Pad2) -> GND_ISO
- T1 pad 10: DC- -> GND_ISO
- T1 pad 11: DC- -> GND_ISO
- T1 pad 12: DC- -> GND_ISO
- T1 pad 13: DC- -> GND_ISO
- T1 pad 14: DC- -> GND_ISO
- T1 pad 22: Net-(P22-Pad1) -> GND_ISO
- T1 pad 9: DC- -> GND_ISO

Commit message: Initial work on inverter card 2 (footprints, layout etc)
Parts:
- added J11: CONN_02X06, Pin_Headers:Pin_Header_Straight_2x06_Pitch2.54mm, F.Cu at (167.4, 121.7)
- added R7: 5, Resistors_THT:R_Axial_DIN0207_L6.3mm_D2.5mm_P7.62mm_Horizontal, F.Cu at (124.5, 55.4)
- C5, C6, C7: moved to F.Cu
- P0, P7: footprint PhoenixContact:MSTBA_25_3p_G_508-1757488 -> Connectors_Phoenix:PhoenixContact_GMSTBA-G_03x7.62mm_Angled
- P1: value CONN_01X03 -> CONN_01X04; footprint PhoenixContact:MSTBA_25_3p_G_508-1757488 -> Connectors_Molex:Molex_KK-6410-04_04x2.54mm_Straight
- P2, P3, P4, P5, P6: footprint PhoenixContact:MSTBA_25_3p_G_508-1757488 -> Connectors_Molex:Molex_KK-6410-04_04x2.54mm_Straight
- R41: footprint Resistors_THT:R_Axial_DIN0414_L11.9mm_D4.5mm_P15.24mm_Horizontal -> Resistors_SMD:R_1206_HandSoldering
- moved TP11 418.6 mm to (77.0, 24.4)
- moved P0 408.9 mm to (68.3, 42.9), turned to 270 degrees
- moved R8 398.4 mm to (86.9, 46.2), turned to 270 degrees
- moved TP12 397.8 mm to (75.9, 132.3)
- moved C52 368.7 mm to (127.8, 124.1)
- moved U30 349.0 mm to (144.5, 109.5), turned to 180 degrees
- moved P4 348.8 mm to (144.5, 46.0)
- moved P5 345.4 mm to (154.2, 30.0)
- moved R9 341.0 mm to (113.8, 109.7), turned to 270 degrees
- moved C42 340.2 mm to (127.8, 128.1)
- moved C1 340.1 mm to (76.5, 49.5), turned to 270 degrees
- moved TP1 338.5 mm to (171.2, 55.6)
- moved C7 328.7 mm to (124.7, 32.0)
- moved P2 318.8 mm to (146.3, 29.5), turned to 180 degrees
- moved TP8 316.2 mm to (187.4, 115.2)
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Connections:
- C7 pad 2: (no net) -> Net-(C7-Pad2)
- U40 pad 6: (no net) -> T-
- U40 pad 7: (no net) -> T+
- U50 pad 6: (no net) -> Net-(J11-Pad4)
- U50 pad 7: (no net) -> Net-(J11-Pad6)
Other:
- copper layers 2 -> 4
- net class DC+ added: clearance 0.5, trace_width 3, via_dia 0.6, via_drill 0.4
- net class UVW added: clearance 0.5, trace_width 4, via_dia 0.6, via_drill 0.4

Commit message: A lot of work on InverterCard 2.0 pcb layout
Parts:
- removed TP1, TP2, TP3, TP4, TP5, TP6: TEST, Measurement_Points:Test_Point
- added G***: LOGO, Switchcraft:Switchcraft_logo_10px_stroke_2000dpi, F.Cu at (227.8, 23.1)
- added REF***: OSHW-Logo2_7.3x6mm_SilkScreen, OpenSourceHardWare:OSHW-Logo2_7.3x6mm_SilkScreen, F.Cu at (240.4, 132.2)
- C11, C12, C13, C14: footprint Capacitors_SMD:C_1206_HandSoldering -> Capacitor_SMD:C_1206_3216Metric_Pad1.42x1.75mm_HandSolder
- C15, C16, C22, C43, C53: footprint Capacitors_SMD:C_1206_HandSoldering -> Capacitor_SMD:C_1206_3216Metric_Pad1.42x1.75mm_HandSolder; moved to B.Cu
- C31, C41, C42, C51, C52: footprint Capacitors_SMD:C_1210_HandSoldering -> Capacitor_SMD:C_1210_3225Metric_Pad1.42x2.65mm_HandSolder; moved to B.Cu
- C5, C6, C7: footprint Capacitors_THT:C_Rect_L19.0mm_W5.0mm_P15.00mm_MKS4 -> Capacitor_THT:C_Rect_L19.0mm_W5.0mm_P15.00mm_MKS4
- CP21: moved to B.Cu
- D21, D31: footprint LEDs:LED_1206_HandSoldering -> LED_SMD:LED_1206_3216Metric_Pad1.42x1.75mm_HandSolder
- J11: footprint Pin_Headers:Pin_Header_Straight_2x06_Pitch2.54mm -> Connector_PinHeader_2.54mm:PinHeader_2x06_P2.54mm_Vertical
- P0, P7: footprint Connectors_Phoenix:PhoenixContact_GMSTBA-G_03x7.62mm_Angled -> Connector_Phoenix_GMSTB:PhoenixContact_GMSTBA_2,5_3-G-7,62_1x03_P7.62mm_Horizontal; moved to B.Cu
- P1: value CONN_01X04 -> CONN_01X03; footprint Connectors_Molex:Molex_KK-6410-04_04x2.54mm_Straight -> Connector_PinHeader_2.54mm:PinHeader_1x03_P2.54mm_Vertical
- P2, P3, P4, P5, P6: footprint Connectors_Molex:Molex_KK-6410-04_04x2.54mm_Straight -> Connector_PinHeader_2.54mm:PinHeader_1x03_P2.54mm_Vertical
- P20: footprint PhoenixContact:MSTBA_25_2p_G_508-1757242 -> Connector_Phoenix_MSTB:PhoenixContact_MSTBA_2,5_2-G-5,08_1x02_P5.08mm_Horizontal
- R1, R2, R3, R4: footprint Resistors_SMD:R_1206_HandSoldering -> Resistor_SMD:R_1206_3216Metric_Pad1.42x1.75mm_HandSolder
- R11, R12, R13, R21, R31, R41, R5, R53, R6: footprint Resistors_SMD:R_1206_HandSoldering -> Resistor_SMD:R_1206_3216Metric_Pad1.42x1.75mm_HandSolder; moved to B.Cu
- R51, R52: footprint Resistors_SMD:R_2010_HandSoldering -> Resistor_SMD:R_1210_3225Metric_Pad1.42x2.65mm_HandSolder; moved to B.Cu
- R7: footprint Resistors_THT:R_Axial_DIN0207_L6.3mm_D2.5mm_P7.62mm_Horizontal -> Resistor_THT:R_Axial_DIN0207_L6.3mm_D2.5mm_P7.62mm_Horizontal
- R8, R9: footprint Resistors_SMD:R_2512_HandSoldering -> Resistor_SMD:R_2512_6332Metric_Pad1.52x3.35mm_HandSolder
- TP10: value TEST -> DC_MID; footprint Measurement_Points:Test_Point -> TestPoint:TestPoint_Loop_D2.50mm_Drill1.0mm_LowProfile
- TP11: value TEST -> DC+; footprint Measurement_Points:Test_Point -> TestPoint:TestPoint_Loop_D2.50mm_Drill1.0mm_LowProfile
- TP12: value TEST -> DC-; footprint Measurement_Points:Test_Point -> TestPoint:TestPoint_Loop_D2.50mm_Drill1.0mm_LowProfile
- TP21: value TEST -> VCC; footprint Measurement_Points:Test_Point -> TestPoint:TestPoint_Loop_D2.50mm_Drill1.0mm_LowProfile
- TP22: value TEST -> GND; footprint Measurement_Points:Test_Point -> TestPoint:TestPoint_Loop_D2.50mm_Drill1.0mm_LowProfile
- TP31: value TEST -> VCC_ISO; footprint Measurement_Points:Test_Point -> TestPoint:TestPoint_Loop_D2.50mm_Drill1.0mm_LowProfile
- TP32: value TEST -> GND_ISO; footprint Measurement_Points:Test_Point -> TestPoint:TestPoint_Loop_D2.50mm_Drill1.0mm_LowProfile
- TP7, TP8, TP9: footprint Measurement_Points:Test_Point -> TestPoint:TestPoint_Loop_D2.50mm_Drill1.0mm_LowProfile
- U30: footprint Housings_DIP:DIP-8_W11.48mm_SMD -> Package_DIP:SMDIP-8_W7.62mm; moved to B.Cu
- U40, U50: footprint Housings_SOIC:SSO-8_6.8x5.9mm_Pitch1.27mm_Clearance8mm -> Package_SO:SSO-8_6.8x5.9mm_P1.27mm_Clearance7mm; moved to B.Cu
- moved TP10 103.0 mm to (96.8, 80.0)
- moved TP7 98.6 mm to (203.9, 32.0)
- moved R51 88.3 mm to (143.6, 112.2), turned to 270 degrees
- moved R2 86.1 mm to (164.0, 57.1), turned to 270 degrees
- moved R41 85.6 mm to (145.8, 126.2), turned to 270 degrees
- moved R1 83.7 mm to (189.2, 50.5)
- moved C16 82.4 mm to (214.1, 55.7), turned to 270 degrees
- moved R4 80.5 mm to (165.4, 75.1)
- moved CP21 79.8 mm to (178.8, 135.1), turned to 270 degrees
- moved C53 76.3 mm to (175.3, 112.8), turned to 90 degrees
- moved R11 75.0 mm to (210.3, 55.6), turned to 270 degrees
- moved R53 75.0 mm to (153.6, 112.2), turned to 270 degrees
- moved P5 74.4 mm to (200.4, 88.3)
- moved C51 70.5 mm to (158.2, 112.2), turned to 270 degrees
- moved C43 69.9 mm to (175.5, 120.9), turned to 270 degrees
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Connections:
- J11 pad 1: VCC -> T+
- J11 pad 10: T- -> Net-(C14-Pad1)
- J11 pad 12: GND -> VCC
- J11 pad 2: GND -> Net-(J11-Pad2)
- J11 pad 3: Net-(C16-Pad1) -> T-
- J11 pad 5: Net-(C15-Pad1) -> GND
- J11 pad 6: Net-(J11-Pad6) -> Net-(C16-Pad1)
- J11 pad 7: Net-(C14-Pad1) -> GND
- J11 pad 8: T+ -> Net-(C15-Pad1)
- U30 pad 8: (no net) -> Net-(U30-Pad8)
- U50 pad 7: Net-(J11-Pad6) -> Net-(J11-Pad2)
Routing:
- net GND: track 0.00 -> 233.3 mm, vias 0 -> 6
- net VCC: track 0.00 -> 231.2 mm
- net GND_ISO: track 0.00 -> 155.5 mm, vias 0 -> 4
- net Net-(C16-Pad1): track 0.00 -> 145.0 mm
- net DC+: track 0.00 -> 116.0 mm, vias 0 -> 1
- net Net-(C15-Pad1): track 0.00 -> 83.0 mm
- net V: track 0.00 -> 79.5 mm, vias 0 -> 1
- net W: track 0.00 -> 65.4 mm, vias 0 -> 2
- net U: track 0.00 -> 63.9 mm, vias 0 -> 2
- net VCC_ISO: track 0.00 -> 59.3 mm
- net Net-(C41-Pad1): track 0.00 -> 57.9 mm, vias 0 -> 1
- net T6_g: track 0.00 -> 36.9 mm, vias 0 -> 1
- net Net-(C51-Pad1): track 0.00 -> 26.8 mm
- net Net-(C14-Pad1): track 0.00 -> 25.1 mm
- net Net-(J11-Pad4): track 0.00 -> 23.8 mm
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- added copper zone on F.Cu, net DC+
- added copper zone on F.Cu, net GND_ISO
- added copper zone on F.Cu, net Net-(C1-Pad2)
- added copper zone on F.Cu, net Net-(P7-Pad1)
- added copper zone on F.Cu, net Net-(P7-Pad2)
- added copper zone on F.Cu, net Net-(P7-Pad3)
- added copper zone on F.Cu, net U
- added copper zone on F.Cu, net V
- added copper zone on F.Cu, net W
Other:
- board outline added: 215 x 126 mm
- net class DC+: trace_width 3 -> 1
- net class UVW: trace_width 4 -> 0.5
- board text added: "1"
- board text added: "11"
- board text added: "12"
- board text added: "2"
- board text added: "DC-Link Voltage Measurement"
- board text added: "GND"
- board text added: "GndISO"
- board text added: "Inverter Board 2.0"
- board text added: "Semikron SKiiP 13ACM12"
- board text added: "T+"
- board text added: "T-"
- board text added: "U"
- board text added: "V"
- board text added: "Vcc"
- board text added: "Vcc OK"
- board text added: "VccISO"
- board text added: "VccIso OK"
- board text added: "W"
- board text added: "dc+"
- board text added: "dc-"
- board text added: "g1"
- board text added: "g2"
- board text added: "g3"
- board text added: "g4"
- board text added: "g5"
- board text added: "g6"
- board text added: "iU"
- board text added: "iV"
- board text added: "iW"
- board text added: "{——GND——}"

Commit message: More adjustments to PCB
Parts:
- C5, C6: value C -> 5uF; footprint Capacitor_THT:C_Rect_L19.0mm_W5.0mm_P15.00mm_MKS4 -> Capacitor_THT:C_Rect_L31.5mm_W11.0mm_P27.50mm_MKS4
- C7: footprint Capacitor_THT:C_Rect_L19.0mm_W5.0mm_P15.00mm_MKS4 -> Capacitor_THT:C_Disc_D6.0mm_W4.4mm_P5.00mm
- CP21: footprint Capacitors_SMD:CP_Elec_6.3x7.7 -> Capacitor_SMD:CP_Elec_6.3x7.7
- R7: footprint Resistor_THT:R_Axial_DIN0207_L6.3mm_D2.5mm_P7.62mm_Horizontal -> Resistor_THT:R_Axial_DIN0617_L17.0mm_D6.0mm_P20.32mm_Horizontal
- TP10, TP11, TP12, TP21, TP22, TP31, TP32, TP7, TP8, TP9: footprint TestPoint:TestPoint_Loop_D2.50mm_Drill1.0mm_LowProfile -> TestPoint:TestPoint_Loop_D2.60mm_Drill1.6mm_Beaded
- U40, U50: footprint Package_SO:SSO-8_6.8x5.9mm_P1.27mm_Clearance7mm -> Package_SO:SSO-8_6.8x5.9mm_P1.27mm_Clearance8mm
- moved C5 17.7 mm to (116.4, 40.7)
- moved R7 12.4 mm to (141.0, 79.9)
- moved C6 4.00 mm to (116.4, 91.7)
- moved G*** 2.88 mm to (225.0, 22.6)
- moved C51 2.29 mm to (158.2, 109.9)
- moved R51 2.29 mm to (143.6, 109.9)
- moved R52 2.29 mm to (148.3, 109.9)
- moved R53 2.29 mm to (153.6, 109.9)
- moved R21 1.94 mm to (207.1, 135.3), turned to 0 degrees
- moved REF*** 1.46 mm to (239.0, 131.7)
- moved C53 1.42 mm to (176.7, 112.7)
- moved C43 1.42 mm to (176.9, 120.8)
Connections:
- J11 pad 11: GND -> VCC
Routing:
- net GND: track 233.3 -> 270.0 mm, vias 6 -> 3
- net VCC: track 231.2 -> 242.2 mm
- net DC+: track 116.0 -> 113.2 mm
- net Net-(C7-Pad2): track 18.5 -> 16.4 mm
- net Net-(C51-Pad1): track 26.8 -> 25.0 mm
- net Net-(C16-Pad1): track 145.0 -> 146.7 mm
- net Net-(C15-Pad1): track 83.0 -> 84.7 mm
- net GND_ISO: track 155.5 -> 154.1 mm
- net T-: track 18.7 -> 17.7 mm
- net VCC_ISO: track 59.3 -> 60.3 mm
- net T+: track 15.7 -> 14.8 mm
Other:
- board text added: "|—GND—|"
- board text removed: "{——GND——}"
